File: Etch-a-sketch/ECE362Project.kicad_sch (KiCad schematic)
At the start: 18 parts, among them J1 USB-Dongle, U2 MMA8451, U3 MPS2202, U4 LM317T

Commit message: updated schematic
Parts:
- R3: value 124 -> 91
- R4: value 174 -> 130
Connections:
- net +3V0: now also U2.6 (VDD); no longer U2.1 (VDD)
- net GND: now also U2.7 (GND); no longer U2.1 (VDD)
- net x_analog: now reaches RV1.2, U1.11 (PA0)
- net y_analog: now reaches RV2.2, U1.12 (PA1)
Changed lines of the file:
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@@
 		)
 	)
+	(label "x_analog"
+		(at 67.31 85.09 0)
+		(fields_autoplaced yes)
+		(effects
+			(font
+				(size 1.27 1.27)
+			)
+			(justify left bottom)
+		)
+	)
+	(label "y_analog"
+		(at 97.79 104.14 0)
+		(fields_autoplaced yes)
+		(effects
+			(font
+				(size 1.27 1.27)
+			)
+			(justify left bottom)
+		)
+	)
 	(global_label "MISO"
 		(shape input)
@@
 			)
 		)
-		(property "Value" "174"
+		(property "Value" "130"
 			(at 93.98 58.4199 0)
 			(effects
@@
 			)
 		)
-		(pin "1"
+		(pin "6"
 		)
 		(pin "2"
@@
 		(pin "1"
 		)
-		(pin "1"
+		(pin "7"
 		)
 		(pin "5"
@@
 			)
 		)
-		(property "Value" "124"
+		(property "Value" "91"
 			(at 93.98 45.7199 0)
 			(effects
