File: Etch-a-sketch/ECE362Project.kicad_sch (KiCad schematic)
At the start: 18 parts, among them J1 USB-Dongle, U2 MMA8451, U3 MPS2202, U4 LM317T

Commit message: updated schematic to include new NRST pullup and adjusted linear regulator resistor values
Parts:
- added R6: 1k, symbol Device:R_US
- R3: value 91 -> 78
Connections:
- net +3V0: now also R6.1
- net at U1.29 (NRST): now also R6.2
- no-connect marks 44 -> 43
Changed lines of the file:
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@@
 	)
 	(no_connect
-		(at 158.75 113.03)
-	)
-	(no_connect
 		(at 189.23 85.09)
 	)
@@
 	(wire
 		(pts
+			(xy 151.13 113.03) (xy 158.75 113.03)
+		)
+		(stroke
+			(width 0)
+			(type default)
+		)
+	)
+	(wire
+		(pts
 			(xy 237.49 41.91) (xy 237.49 43.18)
 		)
@@
 	(wire
 		(pts
+			(xy 151.13 111.76) (xy 151.13 113.03)
+		)
+		(stroke
+			(width 0)
+			(type default)
+		)
+	)
+	(wire
+		(pts
 			(xy 189.23 54.61) (xy 191.77 54.61)
 		)
@@
 	)
 	(symbol
+		(lib_id "Device:R_US")
+		(at 151.13 107.95 0)
+		(unit 1)
+		(exclude_from_sim no)
+		(in_bom yes)
+		(on_board yes)
+		(dnp no)
+		(property "Reference" "R6"
+			(at 146.304 106.68 0)
+			(effects
+				(font
+					(size 1.27 1.27)
+				)
+				(justify left)
+			)
+		)
+		(property "Value" "1k"
+			(at 144.78 109.22 0)
+			(effects
+				(font
+					(size 1.27 1.27)
+				)
+				(justify left)
+			)
+		)
+		(property "Footprint" ""
+			(at 152.146 108.204 90)
+			(effects
+				(font
+					(size 1.27 1.27)
+				)
+				(hide yes)
+			)
+		)
+		(property "Datasheet" "~"
+			(at 151.13 107.95 0)
+			(effects
+				(font
+					(size 1.27 1.27)
+				)
+				(hide yes)
+			)
+		)
+		(property "Description" "Resistor, US symbol"
+			(at 151.13 107.95 0)
+			(effects
+				(font
+					(size 1.27 1.27)
+				)
+				(hide yes)
+			)
+		)
+		(pin "1"
+		)
+		(pin "2"
+		)
+		(instances
+			(project "ECE362Project"
+				(path "/3e4d20ed-557e-4cff-9f91-598a72ef8c78"
+					(reference "R6")
+					(unit 1)
+				)
+			)
+		)
+	)
+	(symbol
 		(lib_id "power:GND")
 		(at 64.77 62.23 0)
@@
 	)
 	(symbol
+		(lib_id "power:+3V0")
+		(at 151.13 104.14 0)
+		(unit 1)
+		(exclude_from_sim no)
+		(in_bom yes)
+		(on_board yes)
+		(dnp no)
+		(property "Reference" "#PWR025"
+			(at 151.13 107.95 0)
+			(effects
+				(font
+					(size 1.27 1.27)
+				)
+				(hide yes)
+			)
+		)
+		(property "Value" "+3V0"
+			(at 149.352 99.06 0)
+			(effects
+				(font
+					(size 1.27 1.27)
+				)
+			)
+		)
+		(property "Footprint" ""
+			(at 151.13 104.14 0)
+			(effects
+				(font
+					(size 1.27 1.27)
+				)
+				(hide yes)
+			)
+		)
+		(property "Datasheet" ""
+			(at 151.13 104.14 0)
+			(effects
+				(font
+					(size 1.27 1.27)
+				)
+				(hide yes)
+			)
+		)
+		(property "Description" "Power symbol creates a global label with name \"+3V0\""
+			(at 151.13 104.14 0)
+			(effects
+				(font
+					(size 1.27 1.27)
+				)
+				(hide yes)
+			)
+		)
+		(pin "1"
+		)
+		(instances
+			(project "ECE362Project"
+				(path "/3e4d20ed-557e-4cff-9f91-598a72ef8c78"
+					(reference "#PWR025")
+					(unit 1)
+				)
+			)
+		)
+	)
+	(symbol
 		(lib_id "Regulator_Linear:LM317_SOT-223")
 		(at 78.74 39.37 0)
@@
 			)
 		)
-		(property "Value" "91"
+		(property "Value" "78"
 			(at 93.98 45.7199 0)
 			(effects
